Commit message: new frame

File: lapy_bot/description/urdf/gazebo_tags.xacro (robot description, xacro)
@@ -7,21 +7,18 @@
   </gazebo>
   <gazebo reference="left_wheel">
-    <!--
     <kp>1000000000000000000000000000.0</kp>
     <kd>1000000000000000000000000000.0</kd>
     <mu1>10.0</mu1>
     <mu2>10.0</mu2>
-    -->
     <material>Gazebo/Blue</material>
   </gazebo>
   <gazebo reference="right_wheel">
-    <!--
     <kp>1000000000000000000000000000.0</kp>
     <kd>1000000000000000000000000000.0</kd>
     <mu1>10.0</mu1>
     <mu2>10.0</mu2>
-    -->
     <material>Gazebo/Blue</material>
   </gazebo>
+<!--
   <gazebo reference="front_caster_wheel">
         <material>Gazebo/White</material>
@@ -29,4 +26,6 @@
         <mu2 value="${caster_wheel_mu2}"/>
     </gazebo>
+-->
+<!--
   <gazebo reference="back_caster_wheel">
         <material>Gazebo/White</material>
@@ -34,3 +33,34 @@
         <mu2 value="${caster_wheel_mu2}"/>
     </gazebo>
+-->
+  <gazebo reference="front_yaw_link">
+      <material>Gazebo/Blue</material>
+  </gazebo>
+  <gazebo reference="front_roll_link">
+        <material>Gazebo/Red</material>
+  </gazebo>
+  <gazebo reference="front_pitch_link">
+    <kp>1000000000000000000000000000.0</kp>
+    <kd>1000000000000000000000000000.0</kd>
+    <mu1>0.5</mu1>
+    <mu2>0.5</mu2>
+    <material>Gazebo/Purple</material>
+  </gazebo>
+  <!-- JOINT PUBLISHER -->
+  <gazebo>
+    <plugin name="lapy_bot_joint_state" filename="libgazebo_ros_joint_state_publisher.so">
+      <ros>
+          <remapping>~/out:=joint_states</remapping>
+      </ros>
+      <update_rate>30</update_rate>
+      <joint_name>left_wheel_joint</joint_name>
+      <joint_name>right_wheel_joint</joint_name>
+      <joint_name>front_yaw_joint</joint_name>
+      <joint_name>back_yaw_joint</joint_name>
+      <joint_name>front_roll_joint</joint_name>
+      <joint_name>back_roll_joint</joint_name>
+      <joint_name>front_pitch_joint</joint_name>
+      <joint_name>back_pitch_joint</joint_name>
+    </plugin>
+  </gazebo>
 </robot>

File: lapy_bot/description/urdf/robot_core.xacro (robot description, xacro)
@@ -9,10 +9,10 @@
     <xacro:property name="chassis_height" value="0.08"/>
     <xacro:property name="chassis_mass" value="1.0"/>
-    <xacro:property name="wheel_radius" value="0.0325"/>
+    <xacro:property name="wheel_radius" value="0.0335"/>  <!-- was 0.0325 before new frame -->
     <xacro:property name="wheel_thickness" value="0.025"/>
     <xacro:property name="wheel_mass" value="0.05"/>
-    <xacro:property name="wheel_offset_x" value="0.115"/>
-    <xacro:property name="wheel_offset_y" value="0.0"/>
-    <xacro:property name="wheel_offset_z" value="0.012"/>
+    <xacro:property name="wheel_offset_x" value="0.045"/>
+    <xacro:property name="wheel_offset_y" value="0.117"/>
+    <xacro:property name="wheel_offset_z" value="0.01425"/>
     <xacro:property name="caster_wheel_radius" value="0.0125"/> <!-- 0.0205 if offset_z = 0-->
     <xacro:property name="caster_wheel_mass" value="0.01"/>
@@ -59,6 +59,8 @@
         <parent link="base_link"/>
         <child link="left_wheel"/>
-        <origin xyz="0 ${wheel_offset_x} ${wheel_offset_z}" rpy="-${pi/2} 0 0" />
+        <origin xyz="${wheel_offset_x} ${wheel_offset_y} ${wheel_offset_z}" rpy="-${pi/2} 0 0" />
         <axis xyz="0 0 1"/>
+        <limit effort="10000" velocity="1000"/>
+        <joint_properties damping="1.0" friction="1.0"/>
     </joint>
     <xacro:wheel_link wheel_name="left_wheel" />
@@ -67,9 +69,11 @@
         <parent link="base_link"/>
         <child link="right_wheel"/>
-        <origin xyz="0 ${-wheel_offset_x} ${wheel_offset_z}" rpy="${pi/2} 0 0" />
+        <origin xyz="${wheel_offset_x} ${-wheel_offset_y} ${wheel_offset_z}" rpy="${pi/2} 0 0" />
         <axis xyz="0 0 -1"/>
+        <limit effort="10000" velocity="1000"/>
+        <joint_properties damping="1.0" friction="1.0"/>
     </joint>
     <xacro:wheel_link wheel_name="right_wheel" />
-    <!-- FRONT CASTER WHEEL -->
+    <!-- FRONT CASTER WHEEL
     <joint name="front_caster_wheel_joint" type="fixed">
         <parent link="chassis"/>
@@ -93,5 +97,6 @@
         </xacro:inertial_sphere>
     </link>
-    <!-- BACK CASTER WHEEL -->
+-->
+    <!-- BACK CASTER WHEEL
     <joint name="back_caster_wheel_joint" type="fixed">
         <parent link="chassis"/>
@@ -115,3 +120,89 @@
         </xacro:inertial_sphere>
     </link>
+    -->
+    <!-- Caster Wheel Front -->
+    <joint name="front_yaw_joint" type="continuous">
+        <origin rpy="0 0 0" xyz="${-caster_wheel_offset_x} 0 ${caster_wheel_offset_z}" />
+        <parent link="chassis" />
+        <child link="front_yaw_link" />
+        <axis xyz="0 0 1" />
+        <limit effort="1000.0" velocity="100.0" />
+        <dynamics damping="0.0" friction="0.1"/>
+    </joint>
+    <link name="front_yaw_link">
+      <visual>
+        <origin rpy="0 1.5707 1.5707" xyz="0 0 0"/>
+        <geometry>
+          <cylinder length="0.001" radius="0.0045000000000000005"/>
+        </geometry>
+        <material name="white"/>
+      </visual>
+      <collision>
+        <origin rpy="0 1.5707 1.5707" xyz="0 0 0"/>
+        <geometry>
+          <cylinder length="0.001" radius="0.0045000000000000005"/>
+        </geometry>
+      </collision>
+      <inertial>
+          <origin rpy="0 1.5707 1.5707" xyz="0 0 0"/>
+          <mass value="0.001"/>
+          <inertia ixx="5.145833333333334e-09" ixy="0" ixz="0" iyy="5.145833333333334e-09" iyz="0" izz="1.0125000000000003e-08"/>
+      </inertial>
+  </link>
+  <joint name="front_roll_joint" type="continuous">
+    <origin rpy="0 0 0" xyz="0 0 0" />
+    <parent link="front_yaw_link" />
+    <child link="front_roll_link" />
+    <axis xyz="1 0 0" />
+    <limit effort="1000.0" velocity="100.0" />
+    <dynamics damping="0.0" friction="0.1"/>
+  </joint>
+  <link name="front_roll_link">
+      <visual>
+        <origin rpy="0 1.5707 1.5707" xyz="0 0 0"/>
+        <geometry>
+          <cylinder length="0.001" radius="0.0045000000000000005"/>
+        </geometry>
+        <material name="white"/>
+      </visual>
+      <collision>
+        <origin rpy="0 1.5707 1.5707" xyz="0 0 0"/>
+        <geometry>
+          <cylinder length="0.001" radius="0.0045000000000000005"/>
+        </geometry>
+      </collision>
+      <inertial>
+          <origin rpy="0 1.5707 1.5707" xyz="0 0 0"/>
+          <mass value="0.001"/>
+          <inertia ixx="5.145833333333334e-09" ixy="0" ixz="0" iyy="5.145833333333334e-09" iyz="0" izz="1.0125000000000003e-08"/>
+      </inertial>
+  </link>
+  <joint name="front_pitch_joint" type="continuous">
+    <origin rpy="0 0 0" xyz="0 0 0" />
+    <parent link="front_roll_link" />
+    <child link="front_pitch_link" />
+    <axis xyz="0 1 0" />
+    <limit effort="1000.0" velocity="100.0" />
+    <dynamics damping="0.0" friction="0.1"/>
+  </joint>
+  <link name="front_pitch_link">
+    <visual>
+      <origin rpy="0 1.5707 1.5707" xyz="0 0 0"/>
+      <geometry>
+        <sphere radius="0.010"/>
+      </geometry>
+      <material name="white"/>
+    </visual>
+    <collision>
+      <origin rpy="0 1.5707 1.5707" xyz="0 0 0"/>
+      <geometry>
+        <sphere radius="0.010"/>
+      </geometry>
+    </collision>
+    <inertial>
+        <origin rpy="0 1.5707 1.5707" xyz="0 0 0"/>
+        <mass value="0.001"/>
+        <inertia ixx="4e-08" ixy="0" ixz="0" iyy="4e-08" iyz="0" izz="4e-08"/>
+    </inertial>
+  </link>
 </robot>
