Commit message: new pkg lapy_mapper and lapy_description

File: lapy_description/urdf/lidar.xacro (robot description, xacro)
@@ -14,5 +14,5 @@
         <visual>
             <geometry>
-                <mesh filename="package://lapy_bot/description/meshes/sensors/rplidar.dae" scale="1.0 1.0 1.0"/>
+                <mesh filename="package://lapy_description/meshes/sensors/rplidar.dae" scale="1.0 1.0 1.0"/>
             </geometry>
         </visual>
@@ -30,5 +30,5 @@
         <sensor name="laser" type="ray">
             <pose> 0 0 0 0 0 0 </pose>
-            <visualize>false</visualize>
+            <visualize>true</visualize>
             <update_rate>10</update_rate>
             <ray>
@@ -42,5 +42,5 @@
                 <range>
                     <min>0.15</min>
-                    <max>12</max>
+                    <max>12.0</max>
                 </range>
             </ray>

File: lapy_description/urdf/lidar_control.xacro (robot description, xacro)
@@ -53,5 +53,5 @@
       <origin rpy="0 0 0" xyz="0 0 0"/>
       <geometry>
-        <mesh filename="package://lapy_bot/description/meshes/sensors/rplidar.dae" scale="1.0 1.0 1.0"/>
+        <mesh filename="package://lapy_description/meshes/sensors/rplidar.dae" scale="1.0 1.0 1.0"/>
       </geometry>
     </visual>
