Commit message: Fix robot z lvl and fix filters

File: lapy_description/urdf/gazebo_tags.xacro (robot description, xacro)
@@ -57,9 +57,9 @@
       <joint_name>right_wheel_joint</joint_name>
       <joint_name>front_yaw_joint</joint_name>
-      <joint_name>back_yaw_joint</joint_name>
+   <!--    <joint_name>back_yaw_joint</joint_name> -->
       <joint_name>front_roll_joint</joint_name>
-      <joint_name>back_roll_joint</joint_name>
+      <!-- <joint_name>back_roll_joint</joint_name> -->
       <joint_name>front_pitch_joint</joint_name>
-      <joint_name>back_pitch_joint</joint_name>
+      <!-- <joint_name>back_pitch_joint</joint_name> -->
     </plugin>
   </gazebo>

File: lapy_description/urdf/link_macros.xacro (robot description, xacro)
@@ -13,5 +13,6 @@
         <collision>
             <geometry>
-                <sphere radius="${wheel_radius}"/>
+                <cylinder radius="${wheel_radius}" length="${wheel_thickness}"/>
+               <!--  <sphere radius="${wheel_radius}"/> -->
             </geometry>
         </collision>

File: lapy_description/urdf/robot.urdf.xacro (robot description, xacro)
@@ -2,4 +2,5 @@
 <robot xmlns:xacro="http://www.ros.org/wiki/xacro"  name="lapyBot">
     <xacro:arg name="use_ros2_control" default="true"/>
+    <xacro:arg name="sim_mode" default="false"/>
     <xacro:include filename="robot_core.xacro" />
      <xacro:if value="$(arg use_ros2_control)">

File: lapy_description/urdf/robot_core.xacro (robot description, xacro)
@@ -134,5 +134,5 @@
         <origin rpy="0 1.5707 1.5707" xyz="0 0 0"/>
         <geometry>
-          <cylinder length="0.001" radius="0.0045000000000000005"/>
+          <sphere radius="${caster_wheel_radius}"/>
         </geometry>
         <material name="white"/>
@@ -141,5 +141,5 @@
         <origin rpy="0 1.5707 1.5707" xyz="0 0 0"/>
         <geometry>
-          <cylinder length="0.001" radius="0.0045000000000000005"/>
+          <sphere radius="${caster_wheel_radius}"/>
         </geometry>
       </collision>
@@ -162,5 +162,5 @@
         <origin rpy="0 1.5707 1.5707" xyz="0 0 0"/>
         <geometry>
-          <cylinder length="0.001" radius="0.0045000000000000005"/>
+          <sphere radius="${caster_wheel_radius}"/>
         </geometry>
         <material name="white"/>
@@ -169,5 +169,5 @@
         <origin rpy="0 1.5707 1.5707" xyz="0 0 0"/>
         <geometry>
-          <cylinder length="0.001" radius="0.0045000000000000005"/>
+          <sphere radius="${caster_wheel_radius}"/>
         </geometry>
       </collision>
@@ -190,5 +190,5 @@
       <origin rpy="0 1.5707 1.5707" xyz="0 0 0"/>
       <geometry>
-        <sphere radius="0.010"/>
+        <sphere radius="${caster_wheel_radius}"/>
       </geometry>
       <material name="white"/>
@@ -197,5 +197,5 @@
       <origin rpy="0 1.5707 1.5707" xyz="0 0 0"/>
       <geometry>
-        <sphere radius="0.010"/>
+        <sphere radius="${caster_wheel_radius}"/>
       </geometry>
     </collision>
